File: hardware/schematics/fake-platka/fake-platka/leg-electronics.kicad_sch (KiCad schematic)
At the start: 21 parts

Commit message: starting to write the documentation
Parts:
- gave numbers to parts that had none: 21
Changed lines of the file:
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@@
   (symbol (lib_id "Device:R") (at 137.16 115.57 0) (unit 1)
     (in_bom yes) (on_board yes) (fields_autoplaced)
-    (property "Reference" "R?" (id 0) (at 139.7 114.2999 0)
+    (property "Reference" "R5" (id 0) (at 139.7 114.2999 0)
       (effects (font (size 1.27 1.27)) (justify left))
     )
@@
   (symbol (lib_id "power:GND") (at 80.01 85.09 0) (unit 1)
     (in_bom yes) (on_board yes) (fields_autoplaced)
-    (property "Reference" "#PWR?" (id 0) (at 80.01 91.44 0)
+    (property "Reference" "#PWR03" (id 0) (at 80.01 91.44 0)
       (effects (font (size 1.27 1.27)) hide)
     )
@@
   (symbol (lib_id "Device:LED") (at 137.16 29.21 180) (unit 1)
     (in_bom yes) (on_board yes) (fields_autoplaced)
-    (property "Reference" "D?" (id 0) (at 138.7475 35.56 0))
+    (property "Reference" "D6" (id 0) (at 138.7475 35.56 0))
     (property "Value" "LED" (id 1) (at 138.7475 33.02 0))
     (property "Footprint" "" (id 2) (at 137.16 29.21 0)
@@
   (symbol (lib_id "Device:Q_Photo_NPN_CE") (at 125.73 60.96 0) (unit 1)
     (in_bom yes) (on_board yes) (fields_autoplaced)
-    (property "Reference" "Q?" (id 0) (at 130.81 58.9406 0)
+    (property "Reference" "Q3" (id 0) (at 130.81 58.9406 0)
       (effects (font (size 1.27 1.27)) (justify left))
     )
@@
   (symbol (lib_id "power:GND") (at 66.04 161.29 0) (unit 1)
     (in_bom yes) (on_board yes) (fields_autoplaced)
-    (property "Reference" "#PWR?" (id 0) (at 66.04 167.64 0)
+    (property "Reference" "#PWR02" (id 0) (at 66.04 167.64 0)
       (effects (font (size 1.27 1.27)) hide)
     )
@@
   (symbol (lib_id "Device:R") (at 149.86 74.93 0) (unit 1)
     (in_bom yes) (on_board yes) (fields_autoplaced)
-    (property "Reference" "R?" (id 0) (at 152.4 73.6599 0)
+    (property "Reference" "R7" (id 0) (at 152.4 73.6599 0)
       (effects (font (size 1.27 1.27)) (justify left))
     )
@@
   (symbol (lib_id "Device:R") (at 69.85 74.93 0) (unit 1)
     (in_bom yes) (on_board yes) (fields_autoplaced)
-    (property "Reference" "R?" (id 0) (at 72.39 73.6599 0)
+    (property "Reference" "R3" (id 0) (at 72.39 73.6599 0)
       (effects (font (size 1.27 1.27)) (justify left))
     )
@@
   (symbol (lib_id "power:GND") (at 66.04 121.92 0) (unit 1)
     (in_bom yes) (on_board yes) (fields_autoplaced)
-    (property "Reference" "#PWR?" (id 0) (at 66.04 128.27 0)
+    (property "Reference" "#PWR01" (id 0) (at 66.04 128.27 0)
       (effects (font (size 1.27 1.27)) hide)
     )
@@
   (symbol (lib_id "power:GND") (at 137.16 123.19 0) (unit 1)
     (in_bom yes) (on_board yes) (fields_autoplaced)
-    (property "Reference" "#PWR?" (id 0) (at 137.16 129.54 0)
+    (property "Reference" "#PWR04" (id 0) (at 137.16 129.54 0)
       (effects (font (size 1.27 1.27)) hide)
     )
@@
   (symbol (lib_id "Device:R") (at 69.85 29.21 90) (unit 1)
     (in_bom yes) (on_board yes) (fields_autoplaced)
-    (property "Reference" "R?" (id 0) (at 69.85 22.86 90))
+    (property "Reference" "R2" (id 0) (at 69.85 22.86 90))
     (property "Value" "150R" (id 1) (at 69.85 25.4 90))
     (property "Footprint" "" (id 2) (at 69.85 30.988 90)
@@
   (symbol (lib_id "Device:Q_Photo_NPN_CE") (at 45.72 60.96 0) (unit 1)
     (in_bom yes) (on_board yes) (fields_autoplaced)
-    (property "Reference" "Q?" (id 0) (at 50.8 58.9406 0)
+    (property "Reference" "Q1" (id 0) (at 50.8 58.9406 0)
       (effects (font (size 1.27 1.27)) (justify left))
     )
@@
   (symbol (lib_id "Device:R") (at 137.16 154.94 0) (unit 1)
     (in_bom yes) (on_board yes) (fields_autoplaced)
-    (property "Reference" "R?" (id 0) (at 139.7 153.6699 0)
+    (property "Reference" "R6" (id 0) (at 139.7 153.6699 0)
       (effects (font (size 1.27 1.27)) (justify left))
     )
@@
   (symbol (lib_id "pspice:DIODE") (at 121.92 151.13 180) (unit 1)
     (in_bom yes) (on_board yes) (fields_autoplaced)
-    (property "Reference" "D?" (id 0) (at 121.92 143.51 0))
+    (property "Reference" "D5" (id 0) (at 121.92 143.51 0))
     (property "Value" "DIODE" (id 1) (at 121.92 146.05 0))
     (property "Footprint" "" (id 2) (at 121.92 151.13 0)
@@
   (symbol (lib_id "Device:Q_Photo_NPN_CE") (at 67.31 55.88 0) (unit 1)
     (in_bom yes) (on_board yes) (fields_autoplaced)
-    (property "Reference" "Q?" (id 0) (at 72.39 53.8606 0)
+    (property "Reference" "Q2" (id 0) (at 72.39 53.8606 0)
       (effects (font (size 1.27 1.27)) (justify left))
     )
@@
   (symbol (lib_id "library:TB67H450AFNG_EL") (at 69.85 104.14 0) (unit 1)
     (in_bom yes) (on_board yes) (fields_autoplaced)
-    (property "Reference" "U?" (id 0) (at 90.17 92.71 0)
+    (property "Reference" "U2" (id 0) (at 90.17 92.71 0)
       (effects (font (size 1.524 1.524)))
     )
@@
   (symbol (lib_id "power:GND") (at 148.59 31.75 0) (unit 1)
     (in_bom yes) (on_board yes) (fields_autoplaced)
-    (property "Reference" "#PWR?" (id 0) (at 148.59 38.1 0)
+    (property "Reference" "#PWR06" (id 0) (at 148.59 38.1 0)
       (effects (font (size 1.27 1.27)) hide)
     )
@@
   (symbol (lib_id "Device:R") (at 128.27 74.93 0) (unit 1)
     (in_bom yes) (on_board yes) (fields_autoplaced)
-    (property "Reference" "R?" (id 0) (at 130.81 73.6599 0)
+    (property "Reference" "R4" (id 0) (at 130.81 73.6599 0)
       (effects (font (size 1.27 1.27)) (justify left))
     )
@@
   (symbol (lib_id "library:TB67H450AFNG_EL") (at 69.85 143.51 0) (unit 1)
     (in_bom yes) (on_board yes) (fields_autoplaced)
-    (property "Reference" "U?" (id 0) (at 90.17 132.08 0)
+    (property "Reference" "U3" (id 0) (at 90.17 132.08 0)
       (effects (font (size 1.524 1.524)))
     )
@@
   (symbol (lib_id "Device:LED") (at 120.65 29.21 180) (unit 1)
     (in_bom yes) (on_board yes) (fields_autoplaced)
-    (property "Reference" "D?" (id 0) (at 122.2375 35.56 0))
+    (property "Reference" "D3" (id 0) (at 122.2375 35.56 0))
     (property "Value" "LED" (id 1) (at 122.2375 33.02 0))
     (property "Footprint" "" (id 2) (at 120.65 29.21 0)
@@
   (symbol (lib_id "Device:Q_Photo_NPN_CE") (at 147.32 55.88 0) (unit 1)
     (in_bom yes) (on_board yes) (fields_autoplaced)
-    (property "Reference" "Q?" (id 0) (at 152.4 53.8606 0)
+    (property "Reference" "Q4" (id 0) (at 152.4 53.8606 0)
       (effects (font (size 1.27 1.27)) (justify left))
     )
@@
   (symbol (lib_id "Device:LED") (at 104.14 29.21 180) (unit 1)
     (in_bom yes) (on_board yes) (fields_autoplaced)
-    (property "Reference" "D?" (id 0) (at 105.7275 35.56 0))
+    (property "Reference" "D2" (id 0) (at 105.7275 35.56 0))
     (property "Value" "LED" (id 1) (at 105.7275 33.02 0))
     (property "Footprint" "" (id 2) (at 104.14 29.21 0)
@@
   (symbol (lib_id "Device:LED") (at 87.63 29.21 180) (unit 1)
     (in_bom yes) (on_board yes) (fields_autoplaced)
-    (property "Reference" "D?" (id 0) (at 89.2175 35.56 0))
+    (property "Reference" "D1" (id 0) (at 89.2175 35.56 0))
     (property "Value" "LED" (id 1) (at 89.2175 33.02 0))
     (property "Footprint" "" (id 2) (at 87.63 29.21 0)
@@
   (symbol (lib_id "pspice:DIODE") (at 121.92 111.76 180) (unit 1)
     (in_bom yes) (on_board yes) (fields_autoplaced)
-    (property "Reference" "D?" (id 0) (at 121.92 104.14 0))
+    (property "Reference" "D4" (id 0) (at 121.92 104.14 0))
     (property "Value" "DIODE" (id 1) (at 121.92 106.68 0))
     (property "Footprint" "" (id 2) (at 121.92 111.76 0)
@@
   (symbol (lib_id "power:GND") (at 137.16 162.56 0) (unit 1)
     (in_bom yes) (on_board yes) (fields_autoplaced)
-    (property "Reference" "#PWR?" (id 0) (at 137.16 168.91 0)
+    (property "Reference" "#PWR05" (id 0) (at 137.16 168.91 0)
       (effects (font (size 1.27 1.27)) hide)
     )
@@
   (symbol (lib_id "power:GND") (at 160.02 85.09 0) (unit 1)
     (in_bom yes) (on_board yes) (fields_autoplaced)
-    (property "Reference" "#PWR?" (id 0) (at 160.02 91.44 0)
+    (property "Reference" "#PWR07" (id 0) (at 160.02 91.44 0)
       (effects (font (size 1.27 1.27)) hide)
     )
@@
   (symbol (lib_id "Device:R") (at 48.26 74.93 0) (unit 1)
     (in_bom yes) (on_board yes) (fields_autoplaced)
-    (property "Reference" "R?" (id 0) (at 50.8 73.6599 0)
+    (property "Reference" "R1" (id 0) (at 50.8 73.6599 0)
       (effects (font (size 1.27 1.27)) (justify left))
     )
@@
   (symbol (lib_id "Motor:Motor_DC") (at 160.02 113.03 0) (mirror x) (unit 1)
     (in_bom yes) (on_board yes) (fields_autoplaced)
-    (property "Reference" "M?" (id 0) (at 154.94 109.2199 0)
+    (property "Reference" "M1" (id 0) (at 154.94 109.2199 0)
       (effects (font (size 1.27 1.27)) (justify right))
     )
@@
   (symbol (lib_id "Motor:Motor_DC") (at 160.02 152.4 0) (mirror x) (unit 1)
     (in_bom yes) (on_board yes) (fields_autoplaced)
-    (property "Reference" "M?" (id 0) (at 154.94 148.5899 0)
+    (property "Reference" "M2" (id 0) (at 154.94 148.5899 0)
       (effects (font (size 1.27 1.27)) (justify right))
     )
