File: hardware/schematics/fake-platka/fake-platka/fake-platka-semi-route.kicad_pcb (KiCad board)
At the start: 2 copper layers, 196.8 x 74.9 mm, 88 parts, among them J1 XT60PW-F, J10 B2B-EH-A, J11 B2B-EH-A, J12 B2B-EH-A, J13 B2B-EH-A, J14 XT60PW-F, J15 XT60PW-F, J16 B2B-EH-A, J17 B2B-EH-A, J18 B2B-EH-A, J19 B2B-EH-A, J2 XT60PW-F, J20 B2B-EH-A, J21 XT60PW-F, J22 XT60PW-F, J23 B2B-EH-A, J24 B2B-EH-A, J25 B2B-EH-A, J26 B2B-EH-A, J27 B2B-EH-A, J28 XT60PW-F, J29 XT60PW-F, J3 B2B-EH-A, J30 B2B-EH-A, J4 B2B-EH-A, J5 B2B-EH-A, J6 B2B-EH-A, J7 XT60PW-F, J8 XT60PW-F, J9 B2B-EH-A, U1 XL4005, U10 TB67H450AFNG_EL, U11 TB67H450AFNG_EL, U12 TB67H450AFNG_EL, U2 XL4005, U3 SC0915-pico-w-board, U4 SC0915-pico-w-board, U5 TB67H450AFNG_EL, U6 TB67H450AFNG_EL, U7 TB67H450AFNG_EL, U8 TB67H450AFNG_EL, U9 TB67H450AFNG_EL

Commit message: working on pcb and documentation
Routing:
- net /Leg Back Left/12V: track 92.0 -> 163.4 mm, vias 1 -> 0
- net /Leg Front Right/FR_F_EB: track 0.00 -> 62.6 mm, vias 0 -> 3
- net /Leg Back Right/BR_F_VREF: track 66.2 -> 12.3 mm, vias 4 -> 1
- net /Leg Front Right/FR_K_EA: track 0.00 -> 53.1 mm
- net Net-(J21-Pad1): track 0.00 -> 51.3 mm, vias 0 -> 3
- net /Leg Front Right/FR_K_EB: track 0.00 -> 49.5 mm
- net Net-(J28-Pad2): track 0.00 -> 41.7 mm, vias 0 -> 2
- net /Leg Front Right/FR_F_EA: track 0.00 -> 39.0 mm, vias 0 -> 1
- net /Left Controller /3V3: track 0.00 -> 34.8 mm
- net Net-(J28-Pad1): track 0.00 -> 33.8 mm, vias 0 -> 2
- net Net-(D7-Pad2): track 0.00 -> 33.0 mm, vias 0 -> 1
- net Net-(J21-Pad2): track 0.00 -> 32.3 mm, vias 0 -> 1
- net Net-(D8-Pad2): track 0.00 -> 30.1 mm
- net Net-(R26-Pad2): track 0.00 -> 23.4 mm, vias 0 -> 2
- net Net-(R23-Pad1): track 0.00 -> 18.4 mm
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