File: hardware/schematics/fake-platka/fake-platka/left_controller.kicad_sch (KiCad schematic)
At the start: 0 parts

Commit message: added all components to the schematic and pcb
Parts:
- added U3: SC0915-pico-w-board, quadruped-lib-footprints:RPi_PicoW_SMD_TH, symbol library:SC0915-pico-w-board
Connections:
- new net 3V3: U3.39 (VSYS)
- new net 3V3_VREF: U3.36 (3V3(OUT))
- new net BL_F_EA: U3.16 (UART0_TX/I2C0_SDA/GPI1_RX/GP12)
- new net BL_F_EB: U3.17 (UART0_RX/I2C0_SCL/SPI1_CSn/GP13)
- new net BL_F_IN1: U3.6 (UART1_TX/I2C0_SDA/SPI0_RX/GP4)
- new net BL_F_IN2: U3.7 (UART1_RX/I2C0_SCL/SPI0_CSn/GP5)
- new net BL_K_EA: U3.19 (I2C1_SDA/SPI1_SCK/GP14)
- new net BL_K_EB: U3.20 (I2C1_SCL/SPI1_TX/GP15)
- new net BL_K_IN1: U3.9 (I2C1_SDA/SPI0_SCK/GP6)
- new net BL_K_IN2: U3.10 (I2C1_SCL/SPI0_TX/GP7)
- new net FL_F_EA: U3.11 (UART1_TX/I2C0_SDA/SPI1_RX/GP8)
- new net FL_F_EB: U3.12 (UART1_RX/I2C0_SCL/SPI1_CSn/GP9)
- new net FL_F_IN1: U3.1 (UART0_TX/I2C0_SDA/SPI0_RX/GP0)
- new net FL_F_IN2: U3.2 (UART0_RX/I2C0_SCL/GPI0_CSn/GP1)
- new net FL_K_EA: U3.14 (I2C1_SDA/SPI1_SCK/GP10)
- new net FL_K_EB: U3.15 (I2C1_SCL/SPI1_TX/GP11)
- new net FL_K_IN1: U3.4 (I2C1_SDA/SPI0_SCK/GP2)
- new net FL_K_IN2: U3.5 (I2C1_SCL/SPI0_TX/GP3)
- new net GND3V3: U3.38 (GND)
- no-connect marks 0 -> 34
Changed lines of the file:
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@@
 (kicad_sch (version 20211123) (generator eeschema)
   (paper "A4")
+  (no_connect (at 212.09 78.74))
+  (no_connect (at 212.09 86.36))
+  (no_connect (at 212.09 114.3))
+  (no_connect (at 212.09 109.22))
+  (no_connect (at 212.09 116.84))
+  (no_connect (at 212.09 121.92))
+  (no_connect (at 85.09 104.14))
+  (no_connect (at 85.09 114.3))
+  (no_connect (at 212.09 83.82))
+  (no_connect (at 212.09 119.38))
+  (no_connect (at 85.09 111.76))
+  (no_connect (at 212.09 111.76))
+  (no_connect (at 85.09 91.44))
+  (no_connect (at 85.09 66.04))
+  (no_connect (at 85.09 121.92))
+  (no_connect (at 212.09 88.9))
+  (no_connect (at 85.09 119.38))
+  (no_connect (at 212.09 127))
+  (no_connect (at 212.09 76.2))
+  (no_connect (at 212.09 60.96))
+  (no_connect (at 212.09 93.98))
+  (no_connect (at 212.09 73.66))
+  (no_connect (at 212.09 124.46))
+  (no_connect (at 212.09 81.28))
+  (no_connect (at 212.09 106.68))
+  (no_connect (at 85.09 78.74))
+  (no_connect (at 212.09 101.6))
+  (no_connect (at 85.09 124.46))
+  (no_connect (at 212.09 71.12))
+  (no_connect (at 212.09 66.04))
+  (no_connect (at 212.09 68.58))
+  (no_connect (at 212.09 63.5))
+  (no_connect (at 85.09 116.84))
+  (no_connect (at 212.09 91.44))
+  (hierarchical_label "GND3V3" (shape output) (at 212.09 99.06 0)
+    (effects (font (size 1.27 1.27)) (justify left))
+  )
+  (hierarchical_label "FL_K_IN1" (shape output) (at 85.09 68.58 180)
+    (effects (font (size 1.27 1.27)) (justify right))
+  )
+  (hierarchical_label "BL_F_IN1" (shape output) (at 85.09 73.66 180)
+    (effects (font (size 1.27 1.27)) (justify right))
+  )
+  (hierarchical_label "3V3_VREF" (shape output) (at 212.09 104.14 0)
+    (effects (font (size 1.27 1.27)) (justify left))
+  )
+  (hierarchical_label "FL_K_IN2" (shape output) (at 85.09 71.12 180)
+    (effects (font (size 1.27 1.27)) (justify right))
+  )
+  (hierarchical_label "FL_F_EB" (shape input) (at 85.09 88.9 180)
+    (effects (font (size 1.27 1.27)) (justify right))
+  )
+  (hierarchical_label "BL_F_EB" (shape input) (at 85.09 101.6 180)
+    (effects (font (size 1.27 1.27)) (justify right))
+  )
+  (hierarchical_label "FL_F_IN1" (shape output) (at 85.09 60.96 180)
+    (effects (font (size 1.27 1.27)) (justify right))
+  )
+  (hierarchical_label "BL_F_EA" (shape input) (at 85.09 99.06 180)
+    (effects (font (size 1.27 1.27)) (justify right))
+  )
+  (hierarchical_label "FL_K_EA" (shape input) (at 85.09 93.98 180)
+    (effects (font (size 1.27 1.27)) (justify right))
+  )
+  (hierarchical_label "FL_F_IN2" (shape output) (at 85.09 63.5 180)
+    (effects (font (size 1.27 1.27)) (justify right))
+  )
+  (hierarchical_label "BL_K_IN1" (shape output) (at 85.09 81.28 180)
+    (effects (font (size 1.27 1.27)) (justify right))
+  )
+  (hierarchical_label "BL_F_IN2" (shape output) (at 85.09 76.2 180)
+    (effects (font (size 1.27 1.27)) (justify right))
+  )
+  (hierarchical_label "FL_F_EA" (shape input) (at 85.09 86.36 180)
+    (effects (font (size 1.27 1.27)) (justify right))
+  )
+  (hierarchical_label "BL_K_IN2" (shape output) (at 85.09 83.82 180)
+    (effects (font (size 1.27 1.27)) (justify right))
+  )
+  (hierarchical_label "3V3" (shape input) (at 212.09 96.52 0)
+    (effects (font (size 1.27 1.27)) (justify left))
+  )
+  (hierarchical_label "FL_K_EB" (shape input) (at 85.09 96.52 180)
+    (effects (font (size 1.27 1.27)) (justify right))
+  )
+  (hierarchical_label "BL_K_EB" (shape input) (at 85.09 109.22 180)
+    (effects (font (size 1.27 1.27)) (justify right))
+  )
+  (hierarchical_label "BL_K_EA" (shape input) (at 85.09 106.68 180)
+    (effects (font (size 1.27 1.27)) (justify right))
+  )
+  (symbol (lib_id "library:SC0915-pico-w-board") (at 85.09 60.96 0) (unit 1)
+    (in_bom yes) (on_board yes) (fields_autoplaced)
+    (property "Reference" "U3" (id 0) (at 148.59 49.53 0)
+      (effects (font (size 1.524 1.524)))
+    )
+    (property "Value" "SC0915-pico-w-board" (id 1) (at 148.59 53.34 0)
+      (effects (font (size 1.524 1.524)))
+    )
+    (property "Footprint" "quadruped-lib-footprints:RPi_PicoW_SMD_TH" (id 2) (at 85.09 60.96 0)
+      (effects (font (size 1.27 1.27) italic) hide)
+    )
+    (property "Datasheet" "SC0915" (id 3) (at 85.09 60.96 0)
+      (effects (font (size 1.27 1.27) italic) hide)
+    )
+    (pin "1")
+    (pin "10")
+    (pin "11")
+    (pin "12")
+    (pin "13")
+    (pin "14")
+    (pin "15")
+    (pin "16")
+    (pin "17")
+    (pin "18")
+    (pin "19")
+    (pin "2")
+    (pin "20")
+    (pin "21")
+    (pin "22")
+    (pin "23")
+    (pin "24")
+    (pin "25")
+    (pin "26")
+    (pin "27")
+    (pin "28")
+    (pin "29")
+    (pin "3")
+    (pin "30")
+    (pin "31")
+    (pin "32")
+    (pin "33")
+    (pin "34")
+    (pin "35")
+    (pin "36")
+    (pin "37")
+    (pin "38")
+    (pin "39")
+    (pin "4")
+    (pin "40")
+    (pin "5")
+    (pin "6")
+    (pin "7")
+    (pin "8")
+    (pin "9")
+    (pin "A")
+    (pin "B")
+    (pin "C")
+    (pin "D")
+    (pin "D1")
+    (pin "D2")
+    (pin "D3")
+    (pin "TP1")
+    (pin "TP2")
+    (pin "TP3")
+    (pin "TP4")
+    (pin "TP5")
+    (pin "TP6")
+  )
 )

Commit message: working on pcb and documentation
Other:
- company: (none) -> By Andrey Shefa
- title: (none) -> First pcb for quadruped robot v3
Changed lines of the file:
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@@
 (kicad_sch (version 20211123) (generator eeschema)
   (paper "A4")
+  (title_block
+    (title "First pcb for quadruped robot v3")
+    (date "2024-02-06")
+    (rev "0")
+    (company "By Andrey Shefa")
+  )
   (no_connect (at 212.09 78.74))
   (no_connect (at 212.09 86.36))
