File: hardware/schematics/fake-platka/fake-platka/leg_bl.kicad_sch (KiCad schematic)
At the start: 0 parts

Commit message: added all components to the schematic and pcb
Parts:
- added D3, D4: 1N4001, Diode_THT:D_DO-41_SOD81_P7.62mm_Horizontal, symbol pspice:DIODE
- added J10, J11, J12, J13, J16: B2B-EH-A, quadruped-lib-footprints:CONN_B2B-EH-A LFSN_JST, symbol library:B2B-EH-A_LFSN
- added J14, J15: XT60PW-F, quadruped-lib-footprints:CONN_XT60PW-F_AMA, symbol library:XT60PW-F
- added R12, R13, R15, R20: 5K, Resistor_THT:R_Axial_DIN0207_L6.3mm_D2.5mm_P10.16mm_Horizontal, symbol Device:R
- added R14: 150R, Resistor_THT:R_Axial_DIN0207_L6.3mm_D2.5mm_P10.16mm_Horizontal, symbol Device:R
- added R16, R17, R18, R19: R1, Resistor_THT:R_Axial_DIN0207_L6.3mm_D2.5mm_P10.16mm_Horizontal, symbol Device:R
- added U7, U8: TB67H450AFNG_EL, quadruped-lib-footprints:P-HSOP8-0405-1.27-002_TOS, symbol library:TB67H450AFNG_EL
Connections:
- new net: R16.1, R18.1, U7.7 (RS)
- new net: D4.2 (A), U8.5 (VM)
- new net: J15.2, U8.6 (OUT1)
- new net: R17.2, R19.2, U8.7 (RS)
- new net: J15.1, U8.8 (OUT2)
- new net: J12.1, R14.1
- new net: D3.2 (A), U7.5 (VM)
- new net: J14.2, U7.6 (OUT1)
- new net: J14.1, U7.8 (OUT2)
- new net 12V: D3.1 (K), D4.1 (K)
- new net 3V3: J10.1, J11.1, J13.1, J16.1, R14.2
- new net BL_F_EA: J11.2, R13.1
- new net BL_F_EB: J10.2, R12.1
- new net BL_F_IN1: U7.3 (IN1)
- new net BL_F_IN2: U7.2 (IN2)
- new net BL_F_VREF: U7.4 (VREF)
- new net BL_K_EA: J16.2, R20.1
- new net BL_K_EB: J13.2, R15.1
- new net BL_K_IN1: U8.3 (IN1)
- new net BL_K_IN2: U8.2 (IN2)
- new net BL_K_VREF: U8.4 (VREF)
- new net GND12V: R16.2, R17.1, R18.2, R19.1, U7.1 (GND), U8.1 (GND)
- new net GND3V3: J12.2, R12.2, R13.2, R15.2, R20.2
Other:
- note added: "3.3/10/0.5"
- note added: "GND is made passive"
- note added: "This is 4 LEDs that are remote"
- note added: "VM is made passive"
- note added: "remote"

Commit message: working on pcb and documentation
Connections:
- net 12V: now also R14.2
- net 3V3: no longer R14.2
- net GND12V: now also J12.2
- net GND3V3: no longer J12.2
Other:
- company: (none) -> By Andrey Shefa
- title: (none) -> First pcb for quadruped robot v3
- moved on the sheet: J10, J11, R12, R13
