File: hardware/schematics/fake-platka/fake-platka/leg_fl.kicad_sch (KiCad schematic)
At the start: 0 parts

Commit message: added all components to the schematic and pcb
Parts:
- added D1, D2: 1N4001, Diode_THT:D_DO-41_SOD81_P7.62mm_Horizontal, symbol pspice:DIODE
- added J3, J4, J5, J6, J9: B2B-EH-A, quadruped-lib-footprints:CONN_B2B-EH-A LFSN_JST, symbol library:B2B-EH-A_LFSN
- added J7, J8: XT60PW-F, quadruped-lib-footprints:CONN_XT60PW-F_AMA, symbol library:XT60PW-F
- added R10, R7, R8, R9: R1, Resistor_THT:R_Axial_DIN0207_L6.3mm_D2.5mm_P10.16mm_Horizontal, symbol Device:R
- added R11, R3, R4, R6: 5K, Resistor_THT:R_Axial_DIN0207_L6.3mm_D2.5mm_P10.16mm_Horizontal, symbol Device:R
- added R5: 150R, Resistor_THT:R_Axial_DIN0207_L6.3mm_D2.5mm_P10.16mm_Horizontal, symbol Device:R
- added U5, U6: TB67H450AFNG_EL, quadruped-lib-footprints:P-HSOP8-0405-1.27-002_TOS, symbol library:TB67H450AFNG_EL
Connections:
- new net: R10.2, R8.2, U6.7 (RS)
- new net: D2.2 (A), U6.5 (VM)
- new net: J8.2, U6.6 (OUT1)
- new net: J8.1, U6.8 (OUT2)
- new net: D1.2 (A), U5.5 (VM)
- new net: J7.2, U5.6 (OUT1)
- new net: R7.1, R9.1, U5.7 (RS)
- new net: J7.1, U5.8 (OUT2)
- new net: J5.1, R5.1
- new net 12V: D1.1 (K), D2.1 (K)
- new net 3V3: J3.1, J4.1, J6.1, J9.1, R5.2
- new net FL_F_EA: J4.2, R4.1
- new net FL_F_EB: J3.2, R3.1
- new net FL_F_IN1: U5.3 (IN1)
- new net FL_F_IN2: U5.2 (IN2)
- new net FL_F_VREF: U5.4 (VREF)
- new net FL_K_EA: J9.2, R11.1
- new net FL_K_EB: J6.2, R6.1
- new net FL_K_IN1: U6.3 (IN1)
- new net FL_K_IN2: U6.2 (IN2)
- new net FL_K_VREF: U6.4 (VREF)
- new net GND12V: R10.1, R7.2, R8.1, R9.2, U5.1 (GND), U6.1 (GND)
- new net GND3V3: J5.2, R11.2, R3.2, R4.2, R6.2
Other:
- note added: "3.3/10/0.5"
- note added: "GND is made passive"
- note added: "This is 4 LEDs that are remote"
- note added: "VM is made passive"
- note added: "remote"

Commit message: working on pcb and documentation
Connections:
- net 12V: now also R5.2
- net 3V3: no longer R5.2
- net GND12V: now also J5.2
- net GND3V3: no longer J5.2
Other:
- company: (none) -> By Andrey Shefa
- title: (none) -> First pcb for quadruped robot v3
- moved on the sheet: J3, J4, R3, R4
