File: hardware/schematics/fake-platka/fake-platka/leg_fr.kicad_sch (KiCad schematic)
At the start: 0 parts

Commit message: added all components to the schematic and pcb
Parts:
- added D5, D6: 1N4001, Diode_THT:D_DO-41_SOD81_P7.62mm_Horizontal, symbol pspice:DIODE
- added J17, J18, J19, J20, J23: B2B-EH-A, quadruped-lib-footprints:CONN_B2B-EH-A LFSN_JST, symbol library:B2B-EH-A_LFSN
- added J21, J22: XT60PW-F, quadruped-lib-footprints:CONN_XT60PW-F_AMA, symbol library:XT60PW-F
- added R21, R22, R24, R29: 5K, Resistor_THT:R_Axial_DIN0207_L6.3mm_D2.5mm_P10.16mm_Horizontal, symbol Device:R
- added R23: 150R, Resistor_THT:R_Axial_DIN0207_L6.3mm_D2.5mm_P10.16mm_Horizontal, symbol Device:R
- added R25, R26, R27, R28: R1, Resistor_THT:R_Axial_DIN0207_L6.3mm_D2.5mm_P10.16mm_Horizontal, symbol Device:R
- added U10, U9: TB67H450AFNG_EL, quadruped-lib-footprints:P-HSOP8-0405-1.27-002_TOS, symbol library:TB67H450AFNG_EL
Connections:
- new net: D5.2 (A), U9.5 (VM)
- new net: D6.2 (A), U10.5 (VM)
- new net: J22.2, U10.6 (OUT1)
- new net: R26.2, R28.2, U10.7 (RS)
- new net: J22.1, U10.8 (OUT2)
- new net: J19.1, R23.1
- new net: J21.1, U9.8 (OUT2)
- new net: J21.2, U9.6 (OUT1)
- new net: R25.1, R27.1, U9.7 (RS)
- new net 12V: D5.1 (K), D6.1 (K)
- new net 3V3: J17.1, J18.1, J20.1, J23.1, R23.2
- new net FR_F_EA: J18.2, R22.1
- new net FR_F_EB: J17.2, R21.1
- new net FR_F_IN1: U9.3 (IN1)
- new net FR_F_IN2: U9.2 (IN2)
- new net FR_F_VREF: U9.4 (VREF)
- new net FR_K_EA: J23.2, R29.1
- new net FR_K_EB: J20.2, R24.1
- new net FR_K_IN1: U10.3 (IN1)
- new net FR_K_IN2: U10.2 (IN2)
- new net FR_K_VREF: U10.4 (VREF)
- new net GND12V: R25.2, R26.1, R27.2, R28.1, U10.1 (GND), U9.1 (GND)
- new net GND3V3: J19.2, R21.2, R22.2, R24.2, R29.2
Other:
- note added: "3.3/10/0.5"
- note added: "GND is made passive"
- note added: "This is 4 LEDs that are remote"
- note added: "VM is made passive"
- note added: "remote"

Commit message: working on pcb and documentation
Connections:
- net 12V: now also R23.2
- net 3V3: no longer R23.2
- net GND12V: now also J19.2
- net GND3V3: no longer J19.2
Other:
- company: (none) -> By Andrey Shefa
- title: (none) -> First pcb for quadruped robot v3
- moved on the sheet: J17, J18, R21, R22
