File: hardware/schematics/fake-platka/fake-platka/right_controller.kicad_sch (KiCad schematic)
At the start: 1 part, among them U4 SC0915-pico-w-board

Commit message: working on pcb and documentation
Other:
- company: (none) -> By Andrey Shefa
- title: (none) -> First pcb for quadruped robot v3
Changed lines of the file:
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@@
 (kicad_sch (version 20211123) (generator eeschema)
   (paper "A4")
+  (title_block
+    (title "First pcb for quadruped robot v3")
+    (date "2024-02-06")
+    (rev "0")
+    (company "By Andrey Shefa")
+  )
   (no_connect (at 213.36 128.27))
   (no_connect (at 213.36 95.25))
