File: hardware/schematics/fake-platka/fake-platka/fake-platka.kicad_pcb (KiCad board)
At the start: 2 copper layers, 196.8 x 74.9 mm, 88 parts, among them J1 XT60PW-F, J10 B2B-EH-A, J11 B2B-EH-A, J12 B2B-EH-A, J13 B2B-EH-A, J14 XT60PW-F, J15 XT60PW-F, J16 B2B-EH-A, J17 B2B-EH-A, J18 B2B-EH-A, J19 B2B-EH-A, J2 XT60PW-F, J20 B2B-EH-A, J21 XT60PW-F, J22 XT60PW-F, J23 B2B-EH-A, J24 B2B-EH-A, J25 B2B-EH-A, J26 B2B-EH-A, J27 B2B-EH-A, J28 XT60PW-F, J29 XT60PW-F, J3 B2B-EH-A, J30 B2B-EH-A, J4 B2B-EH-A, J5 B2B-EH-A, J6 B2B-EH-A, J7 XT60PW-F, J8 XT60PW-F, J9 B2B-EH-A, U1 XL4005, U10 TB67H450AFNG_EL, U11 TB67H450AFNG_EL, U12 TB67H450AFNG_EL, U2 XL4005, U3 SC0915-pico-w-board, U4 SC0915-pico-w-board, U5 TB67H450AFNG_EL, U6 TB67H450AFNG_EL, U7 TB67H450AFNG_EL, U8 TB67H450AFNG_EL, U9 TB67H450AFNG_EL

Commit message: board finished
Parts:
- moved R35 15.3 mm to (203.2, 86.4), turned to 180 degrees
- moved R28 15.3 mm to (203.2, 54.6), turned to 180 degrees
- moved R7 15.3 mm to (67.3, 66.0), turned to 180 degrees
- moved R16 10.9 mm to (67.3, 78.7), turned to 180 degrees
- moved R18 10.9 mm to (67.3, 74.9), turned to 180 degrees
- moved R26 10.9 mm to (203.2, 58.4), turned to 180 degrees
- moved R37 10.8 mm to (203.2, 82.5), turned to 180 degrees
- moved R9 10.8 mm to (67.3, 62.2), turned to 180 degrees
- moved R34 8.25 mm to (193.0, 74.3)
- moved R36 8.25 mm to (193.0, 78.1)
- moved R10 7.66 mm to (57.1, 54.6)
- moved R8 7.66 mm to (57.1, 58.4)
- moved R25 7.62 mm to (193.0, 62.2)
- moved R27 7.62 mm to (193.1, 66.0)
- moved D2 3.39 mm to (102.2, 38.7)
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Routing:
- net /Left Controller /3V3: track 0.00 -> 463.2 mm, vias 0 -> 5
- net /Leg Back Left/12V: track 92.0 -> 539.6 mm, vias 1 -> 15
- net /Left Controller /GND3V3: track 0.00 -> 433.0 mm, vias 0 -> 6
- net /Leg Back Right/GND12V: track 105.9 -> 297.6 mm, vias 4 -> 8
- net /Leg Back Right/BR_K_EB: track 0.00 -> 121.7 mm, vias 0 -> 2
- net /Leg Back Right/BR_K_EA: track 0.00 -> 119.0 mm, vias 0 -> 3
- net /Left Controller /FL_K_EB: track 0.00 -> 95.9 mm, vias 0 -> 2
- net /Left Controller /BL_F_EA: track 0.00 -> 93.6 mm, vias 0 -> 5
- net /Left Controller /FL_K_EA: track 0.00 -> 87.3 mm, vias 0 -> 1
- net /Leg Back Right/BR_F_EA: track 0.00 -> 83.1 mm, vias 0 -> 3
- net /Leg Back Right/BR_F_EB: track 0.00 -> 79.0 mm, vias 0 -> 2
- net /Leg Front Right/FR_K_EB: track 0.00 -> 74.5 mm, vias 0 -> 2
- net /Leg Front Right/FR_K_EA: track 0.00 -> 67.5 mm, vias 0 -> 1
- net /Left Controller /BL_K_EB: track 0.00 -> 65.1 mm, vias 0 -> 3
- net /Leg Front Right/FR_F_EB: track 0.00 -> 65.0 mm, vias 0 -> 2
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
Commit message: finalizing the documentation
Parts:
- moved J23 42.3 mm to (247.5, 72.6)
- moved R21 42.3 mm to (247.5, 96.7)
- moved R23 42.3 mm to (239.9, 98.0)
- moved R25 42.3 mm to (215.7, 98.0)
- moved R28 42.3 mm to (225.9, 90.3)
- moved R29 42.3 mm to (239.9, 90.3)
- moved R30 42.3 mm to (243.7, 114.5)
- moved R32 42.3 mm to (229.7, 114.5)
- moved R33 42.3 mm to (229.7, 118.3)
- moved R35 42.3 mm to (225.9, 122.1)
- moved R36 42.3 mm to (215.7, 113.9)
- moved R37 42.3 mm to (225.9, 118.3)
- moved R38 42.3 mm to (229.7, 122.1)
- moved U10 42.3 mm to (208.1, 92.9)
- moved U12 42.3 mm to (208.1, 119.6)
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Other:
- board size 196.8 x 74.9 mm -> 196.9 x 74.9 mm
